File: Circuit Board/JoeyJoebags.kicad_pcb (KiCad board)
At the start: 2 copper layers, 50 x 50 mm, 6 parts

Commit message: Fix broken footprint for maple mini
Parts:
- Maple Mini: value Maple_Mini -> Maple_Mini_Fixed; footprint Module:Maple_Mini -> Custom:Maple_Mini_Fixed
